File: esp32s2s3dev_custom/esp32s2s3dev_custom.kicad_pcb (KiCad board)
At the start: 2 copper layers, 90 x 75 mm, 33 parts, among them U1 ESP32-S3-DevKitC, U3 R-78E3.3-0.5, U4 L7805

Commit message: add capacitor to registor, regulator to BNO serial
Parts:
- added C2: 0.33u, Capacitor_THT:C_Disc_D3.0mm_W1.6mm_P2.50mm, F.Cu at (170.8, 92.0)
- added C3: 0.1u, Capacitor_THT:C_Disc_D3.0mm_W1.6mm_P2.50mm, F.Cu at (118.5, 92.2)
- added R11: 10k, Resistor_THT:R_Axial_DIN0204_L3.6mm_D1.6mm_P5.08mm_Horizontal, F.Cu at (146.5, 75.8)
- added R12: 10k, Resistor_THT:R_Axial_DIN0204_L3.6mm_D1.6mm_P5.08mm_Horizontal, F.Cu at (143.5, 75.8)
- renumbered GREEN to D1, RED to D2, Vin to J1, Vout to J2
Routing:
- net /BNOTX: track 9.51 -> 23.6 mm, vias 0 -> 2
- net +3V3: track 311.8 -> 325.2 mm, vias 8 -> 9
- net GND: track 362.2 -> 375.5 mm, vias 0 -> 1
- net /BNORX: track 9.49 -> 19.5 mm
- net /SRV1: track 61.1 -> 67.7 mm
- net /SRV2: track 73.6 -> 79.1 mm
- net +5V: track 52.3 -> 57.2 mm, vias 1 -> 2
- net +9V: track 221.9 -> 224.6 mm, vias 0 -> 1
- net /M1IN1: track 72.9 -> 74.8 mm
- net /RO3B: track 77.7 -> 79.0 mm
- net /RO3A: track 71.3 -> 72.4 mm
- net /M1IN2: track 86.0 -> 86.6 mm
- added copper zone on F.Cu, net GND
Other:
- board text added: "0.1u"
- board text added: "0.33u"
- board text added: "12"
- board text added: "1u"
- board text added: "68"
- board text added: "SRV5V"
- board text added: "SRV9.9V"
- board text added: "Vin"
- board text added: "Vout"
